File: robot_chat_PCB/captors.kicad_sch (KiCad schematic)
At the start: 0 parts

Commit message: pcb alim et connecteurs
Parts:
- added J4: Conn_01x08, symbol Connector_Generic:Conn_01x08
- added J5, J6: Conn_01x03, symbol Connector_Generic:Conn_01x03
- added J9: Conn_01x02, symbol Connector_Generic:Conn_01x02
- added JP3, JP4: SolderJumper_2_Bridged, symbol Jumper:SolderJumper_2_Bridged
Connections:
- new net: J4.3 (Pin_3), JP4.2 (B)
- new net: J4.2 (Pin_2), JP3.2 (B)
- new net +3.3V: J5.2 (Pin_2), J6.2 (Pin_2)
- new net +5V: J4.1 (Pin_1)
- new net BACK_BORDER_DETECT: J6.1 (Pin_1)
- new net BUMPER_SW: J9.1 (Pin_1)
- new net FRONT_BORDER_DETECT: J5.1 (Pin_1)
- new net GND: J4.4 (Pin_4), J5.3 (Pin_3), J6.3 (Pin_3), J9.2 (Pin_2)
- new net LIDAR_EN: J4.7 (Pin_7)
- new net LIDAR_RANGING_EN: J4.6 (Pin_6)
- new net LIDAR_RX: JP3.1 (A)
- new net LIDAR_SPEED: J4.5 (Pin_5)
- new net LIDAR_TX: JP4.1 (A)
- no-connect marks 0 -> 1
Other:
- note added: "Bumper"
- note added: "Gsharp"
- note added: "LIDAR"
