File: robot_chat_PCB/captors.kicad_sch (KiCad schematic)
At the start: 9 parts, among them J501 Conn_01x03, J502 Conn_01x08, J503 Conn_01x03, J504 Conn_01x02, U202 LSM6DSM

Commit message: Mise à jour placement
Parts:
- C501, C502: footprint Capacitor_SMD:C_0603_1608Metric -> Capacitor_SMD:C_0402_1005Metric
- D501: value LED_Small -> Bump
- J501: value Conn_01x03 -> F_Detect
- J502: value Conn_01x08 -> Lidar
- J503: value Conn_01x03 -> B_Detect
- J504: value Conn_01x02 -> Bump
Connections:
- net BUMPER_SW: now also R501.2; no longer D501.2 (A)
- net GND: now also D501.1 (K); no longer R501.1
- new net: D501.2 (A), R501.1
Other:
- moved on the sheet: R501
Changed lines of the file:
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@@
     (in_bom yes) (on_board yes) (dnp no)
     (property "Reference" "J503" (at 123.19 144.78 0)
-      (effects (font (size 1.27 1.27)) (justify left))
-    )
-    (property "Value" "Conn_01x03" (at 123.19 147.32 0)
+      (effects (font (size 1.27 1.27)) (justify left) hide)
+    )
+    (property "Value" "B_Detect" (at 123.19 146.05 0)
       (effects (font (size 1.27 1.27)) (justify left))
     )
@@
       (effects (font (size 1.27 1.27)) (justify left))
     )
-    (property "Footprint" "Capacitor_SMD:C_0603_1608Metric" (at 237.49 106.68 0)
+    (property "Footprint" "Capacitor_SMD:C_0402_1005Metric" (at 237.49 106.68 0)
       (effects (font (size 1.27 1.27)) hide)
     )
@@
     )
   )
-  (symbol (lib_id "Device:R_Small") (at 205.74 55.88 180) (unit 1)
-    (in_bom yes) (on_board yes) (dnp no) (fields_autoplaced)
-    (property "Reference" "R501" (at 208.28 54.61 0)
+  (symbol (lib_id "Device:R_Small") (at 205.74 49.53 180) (unit 1)
+    (in_bom yes) (on_board yes) (dnp no) (fields_autoplaced)
+    (property "Reference" "R501" (at 208.28 48.26 0)
       (effects (font (size 1.27 1.27)) (justify right))
     )
-    (property "Value" "1k" (at 208.28 57.15 0)
+    (property "Value" "1k" (at 208.28 50.8 0)
       (effects (font (size 1.27 1.27)) (justify right))
     )
-    (property "Footprint" "Resistor_SMD:R_0603_1608Metric" (at 205.74 55.88 0)
-      (effects (font (size 1.27 1.27)) hide)
-    )
-    (property "Datasheet" "~" (at 205.74 55.88 0)
+    (property "Footprint" "Resistor_SMD:R_0603_1608Metric" (at 205.74 49.53 0)
+      (effects (font (size 1.27 1.27)) hide)
+    )
+    (property "Datasheet" "~" (at 205.74 49.53 0)
       (effects (font (size 1.27 1.27)) hide)
     )
@@
     (in_bom yes) (on_board yes) (dnp no) (fields_autoplaced)
     (property "Reference" "J502" (at 83.82 50.8 0)
-      (effects (font (size 1.27 1.27)) (justify left))
-    )
-    (property "Value" "Conn_01x08" (at 83.82 53.34 0)
+      (effects (font (size 1.27 1.27)) (justify left) hide)
+    )
+    (property "Value" "Lidar" (at 83.82 53.34 0)
       (effects (font (size 1.27 1.27)) (justify left))
     )
@@
   )
   (symbol (lib_id "Connector_Generic:Conn_01x02") (at 222.25 45.72 0) (unit 1)
-    (in_bom yes) (on_board yes) (dnp no) (fields_autoplaced)
+    (in_bom yes) (on_board yes) (dnp no)
     (property "Reference" "J504" (at 224.79 45.72 0)
-      (effects (font (size 1.27 1.27)) (justify left))
-    )
-    (property "Value" "Conn_01x02" (at 224.79 48.26 0)
+      (effects (font (size 1.27 1.27)) (justify left) hide)
+    )
+    (property "Value" "Bump" (at 224.79 46.99 0)
       (effects (font (size 1.27 1.27)) (justify left))
     )
@@
     (in_bom yes) (on_board yes) (dnp no)
     (property "Reference" "J501" (at 66.04 146.05 0)
-      (effects (font (size 1.27 1.27)) (justify left))
-    )
-    (property "Value" "Conn_01x03" (at 66.04 148.59 0)
+      (effects (font (size 1.27 1.27)) (justify left) hide)
+    )
+    (property "Value" "F_Detect" (at 66.04 147.32 0)
       (effects (font (size 1.27 1.27)) (justify left))
     )
@@
       (effects (font (size 1.27 1.27)) (justify left))
     )
-    (property "Footprint" "Capacitor_SMD:C_0603_1608Metric" (at 227.33 106.68 0)
+    (property "Footprint" "Capacitor_SMD:C_0402_1005Metric" (at 227.33 106.68 0)
       (effects (font (size 1.27 1.27)) hide)
     )
@@
     )
   )
-  (symbol (lib_id "Device:LED_Small") (at 205.74 49.53 270) (mirror x) (unit 1)
-    (in_bom yes) (on_board yes) (dnp no)
-    (property "Reference" "D501" (at 203.2 48.1965 90)
+  (symbol (lib_id "Device:LED_Small") (at 205.74 55.88 270) (mirror x) (unit 1)
+    (in_bom yes) (on_board yes) (dnp no)
+    (property "Reference" "D501" (at 203.2 54.5465 90)
+      (effects (font (size 1.27 1.27)) (justify right) hide)
+    )
+    (property "Value" "Bump" (at 203.2 55.88 90)
       (effects (font (size 1.27 1.27)) (justify right))
     )
-    (property "Value" "LED_Small" (at 203.2 50.7365 90)
-      (effects (font (size 1.27 1.27)) (justify right))
-    )
-    (property "Footprint" "LED_SMD:LED_0603_1608Metric" (at 205.74 49.53 90)
-      (effects (font (size 1.27 1.27)) hide)
-    )
-    (property "Datasheet" "~" (at 205.74 49.53 90)
-      (effects (font (size 1.27 1.27)) hide)
-    )
+    (property "Footprint" "LED_SMD:LED_0603_1608Metric" (at 205.74 55.88 90)
+      (effects (font (size 1.27 1.27)) hide)
+    )
+    (property "Datasheet" "~" (at 205.74 55.88 90)
+      (effects (font (size 1.27 1.27)) hide)
+    )

Commit message: changed Rsense position
Parts:
- renumbered J504 to J501, J501 to J504

Commit message: Mise à jour led bumper
Connections:
- net +3.3V: now also J501.1 (Pin_1)
- net BUMPER_SW: now also J501.2 (Pin_2); no longer J501.1 (Pin_1)
- net GND: no longer J501.2 (Pin_2)
Changed lines of the file:
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@@
     (stroke (width 0) (type default))
   )
-  (wire (pts (xy 217.17 48.26) (xy 217.17 50.8))
+  (wire (pts (xy 217.17 40.64) (xy 217.17 43.18))
     (stroke (width 0) (type default))
   )
@@
     )
   )
+  (symbol (lib_id "power:+3.3V") (at 217.17 40.64 0) (unit 1)
+    (in_bom yes) (on_board yes) (dnp no) (fields_autoplaced)
+    (property "Reference" "#PWR0503" (at 217.17 44.45 0)
+      (effects (font (size 1.27 1.27)) hide)
+    )
+    (property "Value" "+3.3V" (at 217.17 35.56 0)
+      (effects (font (size 1.27 1.27)))
+    )
+    (property "Footprint" "" (at 217.17 40.64 0)
+      (effects (font (size 1.27 1.27)) hide)
+    )
+    (property "Datasheet" "" (at 217.17 40.64 0)
+      (effects (font (size 1.27 1.27)) hide)
+    )
+    (pin "1")
+    (instances
+      (project "robot_chat"
+        (path "/74bedd9b-ffd1-4d8b-87e0-848eab324d95/7d20d460-b97c-44b2-b496-8b3ce571e49d"
+          (reference "#PWR0503") (unit 1)
+        )
+      )
+    )
+  )
   (symbol (lib_id "Device:R_Small") (at 205.74 49.53 180) (unit 1)
     (in_bom yes) (on_board yes) (dnp no) (fields_autoplaced)
@@
     )
   )
-  (symbol (lib_id "Connector_Generic:Conn_01x02") (at 222.25 45.72 0) (unit 1)
+  (symbol (lib_id "Connector_Generic:Conn_01x02") (at 222.25 43.18 0) (unit 1)
     (in_bom yes) (on_board yes) (dnp no)
-    (property "Reference" "J501" (at 224.79 45.72 0)
+    (property "Reference" "J501" (at 224.79 43.18 0)
       (effects (font (size 1.27 1.27)) (justify left) hide)
     )
-    (property "Value" "Bump" (at 224.79 46.99 0)
-      (effects (font (size 1.27 1.27)) (justify left))
-    )
-    (property "Footprint" "Connector_JST:JST_XH_S2B-XH-A_1x02_P2.50mm_Horizontal" (at 222.25 45.72 0)
-      (effects (font (size 1.27 1.27)) hide)
-    )
-    (property "Datasheet" "~" (at 222.25 45.72 0)
+    (property "Value" "Bump" (at 224.79 44.45 0)
+      (effects (font (size 1.27 1.27)) (justify left))
+    )
+    (property "Footprint" "Connector_JST:JST_XH_S2B-XH-A_1x02_P2.50mm_Horizontal" (at 222.25 43.18 0)
+      (effects (font (size 1.27 1.27)) hide)
+    )
+    (property "Datasheet" "~" (at 222.25 43.18 0)
       (effects (font (size 1.27 1.27)) hide)
     )
@@
         )
       )
-    )
-  )
-  (symbol (lib_id "power:GND") (at 217.17 50.8 0) (unit 1)
-    (in_bom yes) (on_board yes) (dnp no) (fields_autoplaced)
-    (property "Reference" "#PWR0503" (at 217.17 57.15 0)
-      (effects (font (size 1.27 1.27)) hide)
-    )
-    (property "Value" "GND" (at 217.17 55.88 0)
-      (effects (font (size 1.27 1.27)))
-    )
-    (property "Footprint" "" (at 217.17 50.8 0)
-      (effects (font (size 1.27 1.27)) hide)
-    )
-    (property "Datasheet" "" (at 217.17 50.8 0)
-      (effects (font (size 1.27 1.27)) hide)
-    )
-    (pin "1")
-    (instances
-      (project "robot_chat"
-        (path "/74bedd9b-ffd1-4d8b-87e0-848eab324d95/7d20d460-b97c-44b2-b496-8b3ce571e49d"
-          (reference "#PWR0503") (unit 1)
-        )
-      )

Commit message: fixed DRC, added html bom
Parts:
- D501: Farnell Part Number (none) -> 3796315
- J501: Farnell Part Number (none) -> 1516289
- J502: Farnell Part Number (none) -> 1516296
- J503, J504: Farnell Part Number (none) -> 1516290
- U202: Farnell Part Number (none) -> 2664522
Changed lines of the file:
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@@
+      (effects (font (size 1.27 1.27)) hide)
+    )
+    (property "Farnell Part Number" "2664522" (at 217.17 127 0)
       (effects (font (size 1.27 1.27)) hide)
     )
@@
       (effects (font (size 1.27 1.27)) hide)
     )
+    (property "Farnell Part Number" "1516290" (at 120.65 146.05 0)
+      (effects (font (size 1.27 1.27)) hide)
+    )
     (pin "1")
     (pin "2")
@@
     )
     (property "Datasheet" "~" (at 81.28 50.8 0)
+      (effects (font (size 1.27 1.27)) hide)
+    )
+    (property "Farnell Part Number" "1516296" (at 81.28 50.8 0)
       (effects (font (size 1.27 1.27)) hide)
     )
@@
       (effects (font (size 1.27 1.27)) hide)
     )
+    (property "Farnell Part Number" "1516289" (at 222.25 43.18 0)
+      (effects (font (size 1.27 1.27)) hide)
+    )
     (pin "1")
     (pin "2")
@@
       (effects (font (size 1.27 1.27)) hide)
     )
+    (property "Farnell Part Number" "1516290" (at 63.5 147.32 0)
+      (effects (font (size 1.27 1.27)) hide)
+    )
     (pin "1")
     (pin "2")
@@
       (effects (font (size 1.27 1.27)) hide)
     )
+    (property "Farnell Part Number" "3796315" (at 205.74 55.88 90)
+      (effects (font (size 1.27 1.27)) hide)
+    )
