File: robot_chat_PCB/robot_chat.kicad_sch (KiCad schematic)
At the start: 0 parts

Commit message: Placement composants
Parts:
- added H101, H102, H103, H104: MountingHole_Pad, MountingHole:MountingHole_3.2mm_M3_Pad_Via, symbol Mechanical:MountingHole_Pad
Connections:
- new net GND: H101.1, H102.1, H103.1, H104.1
Changed lines of the file:
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@@
     (company "ENSEA")
   )
+  (junction (at 64.77 109.22) (diameter 0) (color 0 0 0 0)
+  )
+  (junction (at 38.1 109.22) (diameter 0) (color 0 0 0 0)
+  )
   (wire (pts (xy 120.65 104.14) (xy 120.65 115.57))
     (stroke (width 0) (type default))
@@
     (stroke (width 0) (type default))
   )
+  (wire (pts (xy 64.77 109.22) (xy 64.77 111.76))
+    (stroke (width 0) (type default))
+  )
   (wire (pts (xy 82.55 52.07) (xy 102.87 52.07))
     (stroke (width 0) (type default))
   )
+  (wire (pts (xy 38.1 105.41) (xy 38.1 109.22))
+    (stroke (width 0) (type default))
+  )
   (wire (pts (xy 82.55 62.23) (xy 102.87 62.23))
     (stroke (width 0) (type default))
@@
     (stroke (width 0) (type default))
   )
+  (wire (pts (xy 29.21 109.22) (xy 38.1 109.22))
+    (stroke (width 0) (type default))
+  )
   (wire (pts (xy 179.07 50.8) (xy 193.04 50.8))
     (stroke (width 0) (type default))
   )
+  (wire (pts (xy 64.77 105.41) (xy 64.77 109.22))
+    (stroke (width 0) (type default))
+  )
   (wire (pts (xy 118.11 104.14) (xy 118.11 115.57))
     (stroke (width 0) (type default))
@@
     (stroke (width 0) (type default))
   )
+  (wire (pts (xy 38.1 109.22) (xy 38.1 111.76))
+    (stroke (width 0) (type default))
+  )
+  (wire (pts (xy 38.1 109.22) (xy 64.77 109.22))
+    (stroke (width 0) (type default))
+  )
   (wire (pts (xy 140.97 104.14) (xy 140.97 115.57))
     (stroke (width 0) (type default))
@@
     (stroke (width 0) (type default))
   )
+  (symbol (lib_id "Mechanical:MountingHole_Pad") (at 38.1 114.3 180) (unit 1)
+    (in_bom yes) (on_board yes) (dnp no) (fields_autoplaced)
+    (property "Reference" "H103" (at 40.64 114.3 0)
+      (effects (font (size 1.27 1.27)) (justify right))
+    )
+    (property "Value" "MountingHole_Pad" (at 40.64 116.84 0)
+      (effects (font (size 1.27 1.27)) (justify right))
+    )
+    (property "Footprint" "MountingHole:MountingHole_3.2mm_M3_Pad_Via" (at 38.1 114.3 0)
+      (effects (font (size 1.27 1.27)) hide)
+    )
+    (property "Datasheet" "~" (at 38.1 114.3 0)
+      (effects (font (size 1.27 1.27)) hide)
+    )
+    (pin "1")
+    (instances
+      (project "robot_chat"
+        (path "/74bedd9b-ffd1-4d8b-87e0-848eab324d95"
+          (reference "H103") (unit 1)
+        )
+      )
+    )
+  )
+  (symbol (lib_id "Mechanical:MountingHole_Pad") (at 64.77 102.87 0) (unit 1)
+    (in_bom yes) (on_board yes) (dnp no) (fields_autoplaced)
+    (property "Reference" "H102" (at 67.31 100.33 0)
+      (effects (font (size 1.27 1.27)) (justify left))
+    )
+    (property "Value" "MountingHole_Pad" (at 67.31 102.87 0)
+      (effects (font (size 1.27 1.27)) (justify left))
+    )
+    (property "Footprint" "MountingHole:MountingHole_3.2mm_M3_Pad_Via" (at 64.77 102.87 0)
+      (effects (font (size 1.27 1.27)) hide)
+    )
+    (property "Datasheet" "~" (at 64.77 102.87 0)
+      (effects (font (size 1.27 1.27)) hide)
+    )
+    (pin "1")
+    (instances
+      (project "robot_chat"
+        (path "/74bedd9b-ffd1-4d8b-87e0-848eab324d95"
+          (reference "H102") (unit 1)
+        )
+      )
+    )
+  )
+  (symbol (lib_id "power:GND") (at 29.21 109.22 0) (unit 1)
+    (in_bom yes) (on_board yes) (dnp no) (fields_autoplaced)
+    (property "Reference" "#PWR0101" (at 29.21 115.57 0)
+      (effects (font (size 1.27 1.27)) hide)
+    )
+    (property "Value" "GND" (at 29.21 114.3 0)
+      (effects (font (size 1.27 1.27)))
+    )
+    (property "Footprint" "" (at 29.21 109.22 0)
+      (effects (font (size 1.27 1.27)) hide)
+    )
+    (property "Datasheet" "" (at 29.21 109.22 0)
+      (effects (font (size 1.27 1.27)) hide)
+    )
+    (pin "1")
+    (instances
+      (project "robot_chat"
+        (path "/74bedd9b-ffd1-4d8b-87e0-848eab324d95"
+          (reference "#PWR0101") (unit 1)
+        )
+      )
+    )
+  )
+  (symbol (lib_id "Mechanical:MountingHole_Pad") (at 64.77 114.3 180) (unit 1)
+    (in_bom yes) (on_board yes) (dnp no) (fields_autoplaced)
+    (property "Reference" "H104" (at 67.9747 114.3 0)
+      (effects (font (size 1.27 1.27)) (justify right))
+    )
+    (property "Value" "MountingHole_Pad" (at 67.9747 116.84 0)
+      (effects (font (size 1.27 1.27)) (justify right))
+    )
+    (property "Footprint" "MountingHole:MountingHole_3.2mm_M3_Pad_Via" (at 64.77 114.3 0)
+      (effects (font (size 1.27 1.27)) hide)
+    )
+    (property "Datasheet" "~" (at 64.77 114.3 0)
+      (effects (font (size 1.27 1.27)) hide)
+    )
+    (pin "1")
+    (instances
+      (project "robot_chat"
+        (path "/74bedd9b-ffd1-4d8b-87e0-848eab324d95"
+          (reference "H104") (unit 1)
+        )
+      )
+    )
+  )
+  (symbol (lib_id "Mechanical:MountingHole_Pad") (at 38.1 102.87 0) (unit 1)
+    (in_bom yes) (on_board yes) (dnp no) (fields_autoplaced)
+    (property "Reference" "H101" (at 40.64 100.33 0)
+      (effects (font (size 1.27 1.27)) (justify left))
+    )
+    (property "Value" "MountingHole_Pad" (at 40.64 102.87 0)
+      (effects (font (size 1.27 1.27)) (justify left))
+    )
+    (property "Footprint" "MountingHole:MountingHole_3.2mm_M3_Pad_Via" (at 38.1 102.87 0)
+      (effects (font (size 1.27 1.27)) hide)
+    )
+    (property "Datasheet" "~" (at 38.1 102.87 0)
+      (effects (font (size 1.27 1.27)) hide)
+    )
+    (pin "1")
+    (instances
+      (project "robot_chat"
+        (path "/74bedd9b-ffd1-4d8b-87e0-848eab324d95"
+          (reference "H101") (unit 1)
+        )
+      )
+    )
+  )
   (sheet (at 191.77 69.85) (size 43.18 34.29) (fields_autoplaced)
